File: Schematic/Part_C.kicad_sch (KiCad schematic)
At the start: 1 part, among them U9 NUCLEOH723ZG

Commit message: fix nucleo footprint
Parts:
- removed U9: NUCLEOH723ZG, NUCLEOH723ZG:MODULE_NUCLEOH723ZG, symbol NUCLEOH723ZG:NUCLEOH723ZG
