File: Schematic/Schematic.kicad_pcb (KiCad board)
At the start: 2 copper layers, 57 parts, among them J1 Conn_Coaxial, J2 Conn_Coaxial, J3 Conn_Coaxial, J4 Conn_Coaxial, J5 Conn_Coaxial, J6 Conn_Coaxial, J7 USB_C_Receptacle_PowerOnly_6P, U2 MCP1700x-330xxTO, U3 ADA4891-2ARZ-R7, U4 ADA4891-2ARZ-R7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

Commit message: Add updarw
taking a break
Parts:
- moved RV6 162.9 mm to (50.2, 38.1)
Routing:
- net Net-(R4-Pad2): track 1.21 -> 27.6 mm
- net Net-(R5-Pad2): track 0.00 -> 23.6 mm
- net 3V3: track 0.00 -> 21.4 mm
- net Net-(R3-Pad2): track 0.00 -> 16.8 mm
- net Net-(R2-Pad2): track 0.00 -> 12.1 mm
- net pulse_out1: track 0.00 -> 11.5 mm
Changed lines of the file:
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@@
 	(footprint "Potentiometer_THT:Potentiometer_Bourns_3299Y_Vertical"
 		(layer "F.Cu")
-		(at 196.91 108.815)
+		(at 50.165 38.1)
 		(descr "Potentiometer, vertical, Bourns 3299Y, https://www.bourns.com/pdfs/3299.pdf")
 		(tags "Potentiometer vertical Bourns 3299Y")
@@
 	)
 	(segment
+		(start 39.37 55.88)
+		(end 41.91 55.88)
+		(width 0.381)
+		(layer "F.Cu")
+		(net 3)
+	)
+	(segment
+		(start 41.91 55.88)
+		(end 52.07 45.72)
+		(width 0.381)
+		(layer "F.Cu")
+		(net 3)
+	)
+	(segment
+		(start 52.07 45.72)
+		(end 56.5785 45.72)
+		(width 0.381)
+		(layer "F.Cu")
+		(net 3)
+	)
+	(segment
+		(start 61.5315 44.45)
+		(end 65.405 44.45)
+		(width 0.381)
+		(layer "F.Cu")
+		(net 7)
+	)
+	(segment
+		(start 65.405 44.45)
+		(end 67.31 46.355)
+		(width 0.381)
+		(layer "F.Cu")
+		(net 7)
+	)
+	(segment
+		(start 69.85 48.895)
+		(end 67.31 46.355)
+		(width 0.381)
+		(layer "F.Cu")
+		(net 7)
+	)
+	(segment
+		(start 71.755 48.895)
+		(end 69.85 48.895)
+		(width 0.381)
+		(layer "F.Cu")
+		(net 7)
+	)
+	(segment
+		(start 62.865 52.705)
+		(end 64.77 52.705)
+		(width 0.381)
+		(layer "F.Cu")
+		(net 8)
+	)
+	(segment
+		(start 61.5315 48.8315)
+		(end 61.5315 45.72)
+		(width 0.381)
+		(layer "F.Cu")
+		(net 8)
+	)
+	(segment
+		(start 64.77 52.705)
+		(end 67.31 55.245)
+		(width 0.381)
+		(layer "F.Cu")
+		(net 8)
+	)
+	(segment
+		(start 62.865 52.705)
+		(end 62.865 50.165)
+		(width 0.381)
+		(layer "F.Cu")
+		(net 8)
+	)
+	(segment
+		(start 67.31 55.245)
+		(end 67.31 59.055)
+		(width 0.381)
+		(layer "F.Cu")
+		(net 8)
+	)
+	(segment
+		(start 62.865 50.165)
+		(end 61.5315 48.8315)
+		(width 0.381)
+		(layer "F.Cu")
+		(net 8)
+	)
+	(segment
+		(start 47.625 57.15)
+		(end 50.165 54.61)
+		(width 0.381)
+		(layer "F.Cu")
+		(net 9)
+	)
+	(segment
+		(start 50.165 54.61)
+		(end 50.165 52.705)
+		(width 0.381)
+		(layer "F.Cu")
+		(net 9)
+	)
+	(segment
+		(start 55.88 52.705)
+		(end 59.055 49.53)
+		(width 0.381)
+		(layer "F.Cu")
+		(net 9)
+	)
+	(segment
+		(start 50.165 52.705)
+		(end 55.88 52.705)
+		(width 0.381)
+		(layer "F.Cu")
+		(net 9)
+	)
+	(segment
+		(start 59.055 43.18)
+		(end 57.785 41.91)
+		(width 0.381)
+		(layer "F.Cu")
+		(net 9)
+	)
+	(segment
 		(start 57.785 41.91)
 		(end 56.5785 41.91)
@@
 	)
 	(segment
+		(start 59.055 49.53)
+		(end 59.055 43.18)
+		(width 0.381)
+		(layer "F.Cu")
+		(net 9)
+	)
+	(segment
+		(start 45.085 57.15)
+		(end 47.625 57.15)
+		(width 0.381)
+		(layer "F.Cu")
+		(net 9)
+	)
+	(segment
+		(start 53.34 43.0775)
+		(end 56.476 43.0775)
+		(width 0.381)
+		(layer "F.Cu")
+		(net 10)
+	)
+	(segment
+		(start 50.165 38.1)
+		(end 50.165 39.9025)
+		(width 0.381)
+		(layer "F.Cu")
+		(net 10)
+	)
+	(segment
+		(start 39.4725 43.0775)
+		(end 53.34 43.0775)
+		(width 0.381)
+		(layer "F.Cu")
+		(net 10)
+	)
+	(segment
+		(start 56.476 43.0775)
+		(end 56.5785 43.18)
+		(width 0.381)
+		(layer "F.Cu")
+		(net 10)
+	)
+	(segment
+		(start 50.165 39.9025)
+		(end 53.34 43.0775)
+		(width 0.381)
+		(layer "F.Cu")
+		(net 10)
+	)
+	(segment
+		(start 39.37 43.18)
+		(end 39.4725 43.0775)
+		(width 0.381)
+		(layer "F.Cu")
+		(net 10)
+	)
+	(segment
+		(start 45.085 44.45)
+		(end 56.5785 44.45)
+		(width 0.381)
+		(layer "F.Cu")
+		(net 11)
+	)
+	(segment

Commit message: Update
Parts:
- moved U4 155.7 mm to (54.7, 66.7)
Connections:
- U9 pad CN11_28: unconnected-(U9A-PA0-PadCN11_28) -> pulse_out2
- U9 pad CN11_53: unconnected-(U9A-PF0-PadCN11_53) -> pulse_out3
- U9 pad CN11_6: unconnected-(U9A-5V_EXT-PadCN11_6) -> 5V
- U9 pad CN12_11: unconnected-(U9B-PA5-PadCN12_11) -> pulse_out1
- U9 pad CN12_13: unconnected-(U9B-PA6-PadCN12_13) -> pulse_out5
- U9 pad CN12_43: unconnected-(U9B-PD12-PadCN12_43) -> pulse_out6
- U9 pad CN12_62: unconnected-(U9B-PF11-PadCN12_62) -> pulse_out4
Routing:
- net pulse_out1: track 11.5 -> 86.0 mm
- net 3V3: track 21.4 -> 0.00 mm
- net Net-(R4-Pad2): track 27.6 -> 9.24 mm

Commit message: update
Parts:
- D1: footprint LED_THT:LED_D8.0mm -> LED_THT:LED_D3.0mm_Horizontal_O3.81mm_Z2.0mm
- R1: footprint Resistor_THT:R_Axial_DIN0204_L3.6mm_D1.6mm_P5.08mm_Vertical -> Resistor_THT:R_Axial_DIN0309_L9.0mm_D3.2mm_P12.70mm_Horizontal
- moved R8 228.2 mm to (363.9, 151.0), turned to 180 degrees
- moved R9 225.2 mm to (363.4, 144.5), turned to 180 degrees
- moved R10 209.6 mm to (349.8, 137.0)
- moved R13 207.6 mm to (349.8, 130.0)
- moved R14 173.9 mm to (332.6, 69.2)
- moved R15 173.9 mm to (332.6, 73.9)
- moved R16 173.9 mm to (332.6, 78.7)
- moved R17 173.9 mm to (332.6, 83.4)
- moved R18 173.9 mm to (332.6, 88.2)
- moved R19 173.9 mm to (332.6, 92.9)
- moved R20 173.9 mm to (332.6, 97.7)
- moved R21 173.9 mm to (332.6, 102.4)
- moved R23 173.9 mm to (332.6, 107.2)
- moved R25 173.9 mm to (332.6, 111.9)
- moved RV2 173.9 mm to (370.8, 77.1)
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Routing:
- net Net-(R30-Pad2): track 0.00 -> 40.7 mm
- net Net-(J5-In): track 0.00 -> 40.0 mm
- net pulse_out1: track 86.0 -> 115.0 mm
- net Net-(R3-Pad2): track 16.8 -> 44.7 mm
- net Net-(R32-Pad2): track 0.00 -> 25.2 mm
- net Net-(R28-Pad2): track 0.00 -> 22.1 mm
- net Net-(J1-In): track 15.9 -> 36.6 mm
- net Net-(R26-Pad2): track 0.00 -> 17.6 mm
- net pulse_out5: track 0.00 -> 15.0 mm
- net Net-(R5-Pad2): track 23.6 -> 27.8 mm
- net Net-(R4-Pad2): track 9.24 -> 12.4 mm
- net Net-(R2-Pad2): track 12.1 -> 13.1 mm
Other:
- board text removed: "Ethernet"

Commit message: Update PCB
Parts:
- moved R25 275.1 mm to (67.3, 38.7), turned to -90 degrees
- moved R21 263.6 mm to (73.0, 56.5), turned to 90 degrees
- moved R15 252.5 mm to (83.2, 34.3)
- moved RV3 248.8 mm to (125.7, 127.6)
- moved RV5 247.9 mm to (127.6, 51.4)
- moved R20 247.4 mm to (89.5, 51.4), turned to 90 degrees
- moved R17 239.7 mm to (95.9, 45.1), turned to -90 degrees
- moved R10 239.3 mm to (136.5, 28.6)
- moved R9 234.0 mm to (151.8, 44.5)
- moved R33 233.8 mm to (121.9, 44.5)
- moved R37 231.2 mm to (122.6, 62.2)
- moved R8 230.8 mm to (155.6, 51.4), turned to 90 degrees
- moved RV2 217.9 mm to (158.8, 26.7)
- moved R13 217.3 mm to (151.8, 40.6), turned to 180 degrees
- moved R19 209.2 mm to (128.9, 141.0)
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Routing:
- net Net-(R21-Pad2): track 0.00 -> 128.3 mm
- net Net-(J3-In): track 0.00 -> 98.9 mm
- net pulse_out1: track 115.0 -> 25.2 mm
- net Net-(J6-In): track 0.00 -> 47.2 mm
- net Net-(J2-In): track 0.00 -> 43.9 mm
- net Net-(R16-Pad2): track 0.00 -> 42.9 mm
- net Net-(R20-Pad2): track 0.00 -> 37.4 mm
- net Net-(R31-Pad2): track 0.00 -> 34.7 mm
- net Net-(R10-Pad1): track 0.00 -> 34.4 mm
- net Net-(R11-Pad2): track 0.00 -> 33.6 mm
- net Net-(J4-In): track 0.00 -> 31.7 mm
- net Net-(R27-Pad2): track 0.00 -> 29.3 mm
- net Net-(R10-Pad2): track 0.00 -> 26.4 mm
- net pulse_out4: track 0.00 -> 26.1 mm
- net Net-(R19-Pad2): track 0.00 -> 24.0 mm
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
Commit message: Update PCB
Parts:
- J7: footprint Connector_USB:USB_C_Receptacle_GCT_USB4125-xx-x-0190_6P_TopMnt_Horizontal -> Connector_USB:USB_C_Receptacle_GCT_USB4125-xx-x_6P_TopMnt_Horizontal
- U2: footprint Package_TO_SOT_THT:TO-92_Inline -> Package_TO_SOT_THT:TO-92_Inline_Wide
Connections:
- RV4 pad 1: Net-(R32-Pad2) -> GND
- RV4 pad 3: GND -> Net-(R32-Pad2)
- U9 pad CN11_19: Net-(U9A-GND_CN11-PadCN11_19) -> GND
- U9 pad CN11_20: Net-(U9A-GND_CN11-PadCN11_19) -> GND
- U9 pad CN11_22: Net-(U9A-GND_CN11-PadCN11_19) -> GND
- U9 pad CN11_49: Net-(U9A-GND_CN11-PadCN11_19) -> GND
- U9 pad CN11_60: Net-(U9A-GND_CN11-PadCN11_19) -> GND
- U9 pad CN11_8: Net-(U9A-GND_CN11-PadCN11_19) -> GND
- U9 pad CN12_20: Net-(U9B-GND_CN12-PadCN12_20) -> GND
- U9 pad CN12_39: Net-(U9B-GND_CN12-PadCN12_20) -> GND
- U9 pad CN12_54: Net-(U9B-GND_CN12-PadCN12_20) -> GND
- U9 pad CN12_63: Net-(U9B-GND_CN12-PadCN12_20) -> GND
- U9 pad CN12_9: Net-(U9B-GND_CN12-PadCN12_20) -> GND
- U9 pad CN15_1: Net-(U9I-GND_CN15-PadCN15_1) -> GND
- U9 pad CN15_2: Net-(U9I-GND_CN15-PadCN15_1) -> GND
- U9 pad CN16_1: Net-(U9J-GND_CN16-PadCN16_1) -> GND
- U9 pad CN16_2: Net-(U9J-GND_CN16-PadCN16_1) -> GND
- U9 pad CN3_1: Net-(U9G-GND_CN3-PadCN3_1) -> GND
- U9 pad CN3_2: Net-(U9G-GND_CN3-PadCN3_1) -> GND
- U9 pad CN4_1: Net-(U9H-GND_CN4-PadCN4_1) -> GND
- U9 pad CN4_2: Net-(U9H-GND_CN4-PadCN4_1) -> GND
Routing:
- net pulse_out2: track 0.00 -> 164.3 mm
- net 5V: track 0.00 -> 111.9 mm
- net pulse_out6: track 7.58 -> 104.5 mm
- net pulse_out3: track 13.9 -> 110.0 mm
- net pulse_out1: track 25.2 -> 96.8 mm
- net pulse_out5: track 15.0 -> 71.6 mm
- net Net-(D1-A): track 0.00 -> 18.5 mm
- net Net-(J7-CC2): track 0.00 -> 13.0 mm
- net Net-(J1-In): track 36.6 -> 43.9 mm
- net Net-(J5-In): track 42.9 -> 50.0 mm
- net Net-(J7-CC1): track 0.00 -> 5.64 mm
- net Net-(J4-In): track 31.7 -> 36.2 mm
- net GND: track 0.00 -> 3.21 mm
- net Net-(R21-Pad2): track 128.3 -> 129.4 mm
- added copper zone on F.Cu, net 5V
- added copper zone on B.Cu, net GND
- added copper zone on F.Cu, net GND
Other:
- board outline added: 135.3 x 140.3 mm
